File: pcb/kicad/pcb_badge/_autosave-pcb_badge.kicad_pcb (KiCad board)
At the start: 2 copper layers, 82 x 132 mm, 249 parts, among them J1 DEALON USB-TYPE-C-018, J2 Conn_01x02_Pin, J3 Conn_01x04_Pin, J4 Conn_01x03_Pin, J5 Conn_01x03_Pin, J7 Conn_01x02_Pin, Q1 SI2302, Q2 JSM2301S, Q9 2N7002, Q90 2N7002, Q91 2N7002, Q910 2N7002, Q911 2N7002, Q912 2N7002, Q913 2N7002, Q914 2N7002, Q915 2N7002, Q92 2N7002, Q93 2N7002, Q94 2N7002, Q95 2N7002, Q96 2N7002, Q97 2N7002, Q98 2N7002, Q99 2N7002, SW1 SW_MEC_5E, SW2 SW_MEC_5E, SW3 SW_MEC_5E, SW4 SW_MEC_5E, SW5 SW_MEC_5E, SW6 SW_MEC_5E, SW7 SW_MEC_5E, SW8 SW_MEC_5E, U1 TLV70328DBVR, U2 QX2304L33F, U4 74HC238, U8 74HC238, Y1 TAXM8M4RFDCET2T

Commit message: Add battery graphics
Other:
- board text added: "Where to put the battery?"
